File: Design/kicad/Four_Switch_buck_boost/Four_Switch_buck_boost.kicad_sch (KiCad schematic)
At the start: 0 parts

Commit message: no parallel Mosfets and idea to Reduce Cap as per Ripple current
Parts:
- added Q5, Q6, Q7, Q8: Q_NMOS_GDS, Package_TO_SOT_THT:TO-220-3_Vertical, symbol Transistor_FET:Q_NMOS_GDS
- added U1, U2: IR2110, Package_DIP:DIP-14_W7.62mm, symbol Driver_FET:IR2110
Connections:
- no-connect marks 0 -> 1
Other:
- added sheet Sensing and Controller (sensor_and_controller.kicad_sch)
- note added: "Gate Driver"

Commit message: initiated LTspice turns out need to wound own Inductor
Parts:
- added L1: L, symbol Device:L
Other:
- moved on the sheet: Q5, Q6, Q7, Q8, U1, U2
Changed lines of the file:
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@@
 	(paper "A4")
 	(rectangle
-		(start 13.97 90.17)
-		(end 158.75 194.31)
+		(start -182.88 63.5)
+		(end -38.1 167.64)
 		(stroke
 			(width 0)
@@
 	(text "Gate Driver"
 		(exclude_from_sim no)
-		(at 24.892 82.296 0)
+		(at -171.958 55.626 0)
 		(effects
 			(font
@@
 	)
 	(image
-		(at 49.53 106.68)
+		(at -147.32 80.01)
 		(data "iVBORw0KGgoAAAANSUhEUgAAAxcAAAFSCAIAAAAPSLWdAAAAA3NCSVQICAjb4U/gAAAgAElEQVR4"
 			"nOzdeSBU3/84/jv2fSm77NpE9pIUolBoe5VCRYRKpZTSJlq0qLTvoUIR7YtKJNIiS6IFWUJk3/eZ"
@@
 	(symbol
 		(lib_id "Transistor_FET:Q_NMOS_GDS")
-		(at 185.42 93.98 0)
+		(at 124.46 68.58 0)
 		(unit 1)
 		(body_style 1)
@@
 		(fields_autoplaced yes)
 		(property "Reference" "Q5"
-			(at 191.77 92.7099 0)
+			(at 130.81 67.3099 0)
 			(show_name no)
 			(do_not_autoplace no)
@@
 		)
 		(property "Value" "Q_NMOS_GDS"
-			(at 191.77 95.2499 0)
+			(at 130.81 69.8499 0)
 			(show_name no)
 			(do_not_autoplace no)
@@
 		)
 		(property "Footprint" "Package_TO_SOT_THT:TO-220-3_Vertical"
-			(at 190.5 91.44 0)
+			(at 129.54 66.04 0)
 			(hide yes)
 			(show_name no)
@@
 		)
 		(property "Datasheet" ""
-			(at 185.42 93.98 0)
+			(at 124.46 68.58 0)
 			(hide yes)
 			(show_name no)
@@
 		)
 		(property "Description" "N-MOSFET transistor, gate/drain/source"
-			(at 185.42 93.98 0)
+			(at 124.46 68.58 0)
 			(hide yes)
 			(show_name no)
@@
 	(symbol
 		(lib_id "Driver_FET:IR2110")
-		(at 120.65 138.43 90)
+		(at -76.2 111.76 90)
 		(unit 1)
 		(body_style 1)
@@
 		(fields_autoplaced yes)
 		(property "Reference" "U1"
-			(at 105.41 132.9846 90)
+			(at -91.44 106.3146 90)
 			(show_name no)
 			(do_not_autoplace no)
@@
 		)
 		(property "Value" "IR2110"
-			(at 105.41 135.5246 90)
+			(at -91.44 108.8546 90)
 			(show_name no)
 			(do_not_autoplace no)
@@
 		)
 		(property "Footprint" "Package_DIP:DIP-14_W7.62mm"
-			(at 120.65 138.43 0)
+			(at -76.2 111.76 0)
 			(hide yes)
 			(show_name no)
@@
 		)
 		(property "Datasheet" "https://www.infineon.com/dgdl/ir2110.pdf?fileId=5546d462533600a4015355c80333167e"
-			(at 120.65 138.43 0)
+			(at -76.2 111.76 0)
 			(hide yes)
 			(show_name no)
@@
 		)
 		(property "Description" "High and Low Side Driver, 500V, 2.0/2.0A, PDIP-14"
-			(at 120.65 138.43 0)
+			(at -76.2 111.76 0)
 			(hide yes)
 			(show_name no)
@@
 	(symbol
 		(lib_id "Transistor_FET:Q_NMOS_GDS")
-		(at 185.42 107.95 0)
+		(at 124.46 109.22 0)
 		(unit 1)
 		(body_style 1)
@@
 		(fields_autoplaced yes)
 		(property "Reference" "Q6"
-			(at 191.77 106.6799 0)
+			(at 130.81 107.9499 0)
 			(show_name no)
 			(do_not_autoplace no)
@@
 		)
 		(property "Value" "Q_NMOS_GDS"
-			(at 191.77 109.2199 0)
+			(at 130.81 110.4899 0)
 			(show_name no)
 			(do_not_autoplace no)
@@
 		)
 		(property "Footprint" "Package_TO_SOT_THT:TO-220-3_Vertical"
-			(at 190.5 105.41 0)
+			(at 129.54 106.68 0)
 			(hide yes)
 			(show_name no)
@@
 		)
 		(property "Datasheet" ""
-			(at 185.42 107.95 0)
+			(at 124.46 109.22 0)
 			(hide yes)
 			(show_name no)
@@
 		)
 		(property "Description" "N-MOSFET transistor, gate/drain/source"
-			(at 185.42 107.95 0)
+			(at 124.46 109.22 0)
 			(hide yes)
 			(show_name no)
@@
 	(symbol
 		(lib_id "Driver_FET:IR2110")
-		(at 53.34 168.91 90)
+		(at -143.51 142.24 90)
 		(unit 1)
 		(body_style 1)
@@
 		(fields_autoplaced yes)
 		(property "Reference" "U2"
-			(at 38.1 163.4646 90)
+			(at -158.75 136.7946 90)
 			(show_name no)
 			(do_not_autoplace no)
@@
 		)
 		(property "Value" "IR2110"
-			(at 38.1 166.0046 90)
+			(at -158.75 139.3346 90)
 			(show_name no)
 			(do_not_autoplace no)
@@
 		)
 		(property "Footprint" "Package_DIP:DIP-14_W7.62mm"
-			(at 53.34 168.91 0)
+			(at -143.51 142.24 0)
 			(hide yes)
 			(show_name no)
@@
 		)
 		(property "Datasheet" "https://www.infineon.com/dgdl/ir2110.pdf?fileId=5546d462533600a4015355c80333167e"
-			(at 53.34 168.91 0)
+			(at -143.51 142.24 0)
 			(hide yes)
 			(show_name no)
@@
 		)
 		(property "Description" "High and Low Side Driver, 500V, 2.0/2.0A, PDIP-14"
-			(at 53.34 168.91 0)
+			(at -143.51 142.24 0)
 			(hide yes)
 			(show_name no)
@@
 	)
 	(symbol
+		(lib_id "Device:L")
+		(at 152.4 88.9 90)
+		(unit 1)
+		(body_style 1)
+		(exclude_from_sim no)
+		(in_bom yes)
+		(on_board yes)
+		(in_pos_files yes)
+		(dnp no)
+		(fields_autoplaced yes)
+		(property "Reference" "L1"
+			(at 152.4 83.82 90)
+			(show_name no)
+			(do_not_autoplace no)
+			(effects
+				(font
+					(size 1.27 1.27)
+				)
+			)
+		)
+		(property "Value" "L"
+			(at 152.4 86.36 90)
+			(show_name no)
+			(do_not_autoplace no)
+			(effects
+				(font
+					(size 1.27 1.27)
+				)
+			)
+		)
+		(property "Footprint" ""
+			(at 152.4 88.9 0)
+			(hide yes)
+			(show_name no)
+			(do_not_autoplace no)
+			(effects
+				(font
+					(size 1.27 1.27)
+				)
+			)
+		)
+		(property "Datasheet" ""
+			(at 152.4 88.9 0)
+			(hide yes)
+			(show_name no)
+			(do_not_autoplace no)
+			(effects
+				(font
+					(size 1.27 1.27)
+				)
+			)
+		)
+		(property "Description" "Inductor"
+			(at 152.4 88.9 0)
+			(hide yes)
+			(show_name no)
+			(do_not_autoplace no)
+			(effects
+				(font
+					(size 1.27 1.27)
+				)
+			)
+		)
+		(pin "2"
+		)
+		(pin "1"
+		)
+		(instances
+			(project "Four_Switch_buck_boost"
+				(path "/c7b8504e-f9c7-4ff1-8cae-9ccbedfcfbe6"
+					(reference "L1")
+					(unit 1)
+				)
+			)
+		)
+	)
+	(symbol
 		(lib_id "Transistor_FET:Q_NMOS_GDS")
-		(at 214.63 107.95 0)
+		(at 175.26 109.22 0)
 		(unit 1)
 		(body_style 1)
@@
 		(fields_autoplaced yes)
 		(property "Reference" "Q8"
-			(at 220.98 106.6799 0)
+			(at 181.61 107.9499 0)
 			(show_name no)
 			(do_not_autoplace no)
@@
 		)
 		(property "Value" "Q_NMOS_GDS"
-			(at 220.98 109.2199 0)
+			(at 181.61 110.4899 0)
 			(show_name no)
 			(do_not_autoplace no)
@@
 		)
 		(property "Footprint" "Package_TO_SOT_THT:TO-220-3_Vertical"
-			(at 219.71 105.41 0)
+			(at 180.34 106.68 0)
 			(hide yes)
 			(show_name no)
@@
 		)
 		(property "Datasheet" ""
-			(at 214.63 107.95 0)
+			(at 175.26 109.22 0)
 			(hide yes)
 			(show_name no)
@@
 		)
 		(property "Description" "N-MOSFET transistor, gate/drain/source"
-			(at 214.63 107.95 0)
+			(at 175.26 109.22 0)
 			(hide yes)
 			(show_name no)
@@
 	(symbol
 		(lib_id "Transistor_FET:Q_NMOS_GDS")
-		(at 214.63 93.98 0)
+		(at 175.26 68.58 0)
 		(unit 1)
 		(body_style 1)
@@
 		(fields_autoplaced yes)
 		(property "Reference" "Q7"
-			(at 220.98 92.7099 0)
+			(at 181.61 67.3099 0)
 			(show_name no)
 			(do_not_autoplace no)
@@
 		)
 		(property "Value" "Q_NMOS_GDS"
-			(at 220.98 95.2499 0)
+			(at 181.61 69.8499 0)
 			(show_name no)
 			(do_not_autoplace no)
@@
 		)
 		(property "Footprint" "Package_TO_SOT_THT:TO-220-3_Vertical"
-			(at 219.71 91.44 0)
+			(at 180.34 66.04 0)
 			(hide yes)
 			(show_name no)
@@
 		)
 		(property "Datasheet" ""
-			(at 214.63 93.98 0)
+			(at 175.26 68.58 0)
 			(hide yes)
 			(show_name no)
@@
 		)
 		(property "Description" "N-MOSFET transistor, gate/drain/source"
-			(at 214.63 93.98 0)
-			(hide yes)
-			(show_name no)
+			(at 175.26 68.58 0)
+			(hide yes)
+			(show_name no)
